Commit message: urdf modified. still needs new body mesh

File: turtlebot3_description/urdf/turtlebot3_burger.urdf.xacro (robot description, xacro)
@@ -13,5 +13,5 @@
       <origin xyz="-0.032 0 0.0" rpy="0 0 0"/>
       <geometry>
-        <mesh filename="package://turtlebot3_description/meshes/bases/burger_base.stl" scale="0.001 0.001 0.001"/>
+        <mesh filename="package://turtlebot3_description/meshes/bases/burger_base.stl" scale="0.001 0.001 0.005"/>
       </geometry>
       <material name="light_black"/>
@@ -142,5 +142,5 @@
   <!-- Camera -->
   <joint type="fixed" name="camera_joint">
-    <origin xyz="0.03 0 0.11" rpy="0 0.79 0"/>
+    <origin xyz="-0.03 0 0.81" rpy="0 -1.5708 0"/>
     <child link="camera_link"/>
     <parent link="base_link"/>
