Commit message: backup from my f*d up linux

File: urdf/turtlebot3_burger.gazebo.xacro (robot description, xacro)
@@ -4,5 +4,5 @@
   <xacro:arg name="imu_visual"   default="false"/>
   <gazebo reference="base_link">
-    <material>Gazebo/DarkGrey</material>
+    <material>Gazebo/LightGrey</material>
   </gazebo>
   <gazebo reference="wheel_left_link">
@@ -58,5 +58,5 @@
       <rightJoint>wheel_right_joint</rightJoint>
       <wheelSeparation>0.160</wheelSeparation>
-      <wheelDiameter>0.066</wheelDiameter>
+      <wheelDiameter>0.165</wheelDiameter>
       <wheelAcceleration>1</wheelAcceleration>
       <wheelTorque>10</wheelTorque>

File: urdf/turtlebot3_burger.urdf.xacro (robot description, xacro)
@@ -2,5 +2,5 @@
 <robot name="turtlebot3_burger" xmlns:xacro="http://ros.org/wiki/xacro">
   <xacro:include filename="$(find turtlebot3_description)/urdf/common_properties.xacro"/>
-  <xacro:include filename="$(find koghf)/turtlebot3_description/urdf/turtlebot3_burger.gazebo.xacro"/>
+  <xacro:include filename="$(find koghf)/urdf/turtlebot3_burger.gazebo.xacro"/>
   <link name="base_footprint"/>
   <joint name="base_joint" type="fixed">
@@ -11,14 +11,14 @@
   <link name="base_link">
     <visual>
-      <origin xyz="-0.032 0 0.0" rpy="0 0 0"/>
+      <origin xyz="0 0 0.57" rpy="0 0 0"/>
       <geometry>
-        <mesh filename="package://turtlebot3_description/meshes/bases/burger_base.stl" scale="0.001 0.001 0.005"/>
+        <cylinder length="1" radius="0.23"/>
       </geometry>
-      <material name="light_black"/>
+      <material name="green"/>
     </visual>
     <collision>
-      <origin xyz="-0.032 0 0.070" rpy="0 0 0"/>
+      <origin xyz=" 0 0.570" rpy="0 0 0"/>
       <geometry>
-        <box size="0.140 0.140 0.143"/>
+        <cylinder length="1" radius="0.23"/>
       </geometry>
     </collision>
@@ -34,5 +34,5 @@
     <parent link="base_link"/>
     <child link="wheel_left_link"/>
-    <origin xyz="0.0 0.08 0.023" rpy="-1.57 0 0"/>
+    <origin xyz="0.0 0.2 0.165" rpy="-1.57 0 0"/>
     <axis xyz="0 0 1"/>
   </joint>
@@ -41,5 +41,5 @@
       <origin xyz="0 0 0" rpy="1.57 0 0"/>
       <geometry>
-        <mesh filename="package://turtlebot3_description/meshes/wheels/left_tire.stl" scale="0.001 0.001 0.001"/>
+        <mesh filename="package://turtlebot3_description/meshes/wheels/left_tire.stl" scale="0.005 0.005 0.005"/>
       </geometry>
       <material name="dark"/>
@@ -48,5 +48,5 @@
       <origin xyz="0 0 0" rpy="0 0 0"/>
       <geometry>
-        <cylinder length="0.018" radius="0.033"/>
+        <cylinder length="0.09" radius="0.165"/>
       </geometry>
     </collision>
@@ -62,5 +62,5 @@
     <parent link="base_link"/>
     <child link="wheel_right_link"/>
-    <origin xyz="0.0 -0.080 0.023" rpy="-1.57 0 0"/>
+    <origin xyz="0.0 -0.20 0.165" rpy="-1.57 0 0"/>
     <axis xyz="0 0 1"/>
   </joint>
@@ -69,5 +69,5 @@
       <origin xyz="0 0 0" rpy="1.57 0 0"/>
       <geometry>
-        <mesh filename="package://turtlebot3_description/meshes/wheels/right_tire.stl" scale="0.001 0.001 0.001"/>
+        <mesh filename="package://turtlebot3_description/meshes/wheels/right_tire.stl" scale="0.005 0.005 0.005"/>
       </geometry>
       <material name="dark"/>
@@ -76,5 +76,5 @@
       <origin xyz="0 0 0" rpy="0 0 0"/>
       <geometry>
-        <cylinder length="0.018" radius="0.033"/>
+        <cylinder length="0.019" radius="0.165"/>
       </geometry>
     </collision>
@@ -90,5 +90,5 @@
     <parent link="base_link"/>
     <child link="caster_back_link"/>
-    <origin xyz="-0.081 0 -0.004" rpy="-1.57 0 0"/>
+    <origin xyz="-0.281 0 -0.004" rpy="-1.57 0 0"/>
   </joint>
   <link name="caster_back_link">
@@ -96,5 +96,5 @@
       <origin xyz="0 0.001 0" rpy="0 0 0"/>
       <geometry>
-        <box size="0.030 0.009 0.020"/>
+        <box size="0.050 0.02 0.040"/>
       </geometry>
     </collision>
@@ -142,5 +142,5 @@
   <!-- Camera -->
   <joint type="fixed" name="camera_joint">
-    <origin xyz="-0.03 0 0.81" rpy="0 -1.5708 0"/>
+    <origin xyz="-0.03 0 1.1" rpy="0 -1.5708 0"/>
     <child link="camera_link"/>
     <parent link="base_link"/>

Commit message: NOT YEEEEEEEEEEEEETgit add .!

File: urdf/turtlebot3_burger.gazebo.xacro (robot description, xacro)
@@ -4,9 +4,12 @@
   <xacro:arg name="imu_visual"   default="false"/>
   <gazebo reference="base_link">
+    <material>Gazebo/Grey</material>
+  </gazebo>
+  <gazebo reference="tray_link">
     <material>Gazebo/DarkGrey</material>
   </gazebo>
   <gazebo reference="wheel_left_link">
-    <mu1>0.1</mu1>
-    <mu2>0.1</mu2>
+    <mu1>50</mu1>
+    <mu2>50</mu2>
     <kp>500000.0</kp>
     <kd>10.0</kd>
@@ -17,6 +20,6 @@
   </gazebo>
   <gazebo reference="wheel_right_link">
-    <mu1>0.1</mu1>
-    <mu2>0.1</mu2>
+    <mu1>50</mu1>
+    <mu2>50</mu2>
     <kp>500000.0</kp>
     <kd>10.0</kd>
@@ -27,11 +30,11 @@
   </gazebo>
   <gazebo reference="caster_back_link">
-    <mu1>0.1</mu1>
-    <mu2>0.1</mu2>
+    <mu1>0.01</mu1>
+    <mu2>0.01</mu2>
     <kp>1000000.0</kp>
     <kd>100.0</kd>
     <minDepth>0.001</minDepth>
     <maxVel>1.0</maxVel>
-    <material>Gazebo/FlatBlack</material>
+    <material>Gazebo/</material>
   </gazebo>
   <gazebo reference="imu_link">
@@ -54,10 +57,10 @@
       <publishWheelJointState>true</publishWheelJointState>
       <legacyMode>false</legacyMode>
-      <updateRate>30</updateRate>
+      <updateRate>600</updateRate>
       <leftJoint>wheel_left_joint</leftJoint>
       <rightJoint>wheel_right_joint</rightJoint>
-      <wheelSeparation>0.160</wheelSeparation>
-      <wheelDiameter>0.066</wheelDiameter>
-      <wheelAcceleration>1</wheelAcceleration>
+      <wheelSeparation>0.46</wheelSeparation>
+      <wheelDiameter>0.33</wheelDiameter>
+      <wheelAcceleration>3</wheelAcceleration>
       <wheelTorque>10</wheelTorque>
       <rosDebugLevel>na</rosDebugLevel>
@@ -140,13 +143,6 @@
           <far>10.0</far>
         </clip>
-        <noise>
-          <type>gaussian</type>
-          <!-- Noise is sampled independently per pixel on each frame.
-               That pixel's noise value is added to each of its color
-               channels, which at that point lie in the range [0,1]. -->
-          <mean>0.0</mean>
-          <stddev>0.007</stddev>
-        </noise>
       </camera>
+      <visualise>true</visualise>
       <plugin name="camera_controller" filename="libgazebo_ros_camera.so">
         <alwaysOn>true</alwaysOn>

File: urdf/turtlebot3_burger.xacro (robot description, xacro)
@@ -3,30 +3,29 @@
   <xacro:include filename="$(find koghf)/urdf/common_properties.xacro"/>
   <xacro:include filename="$(find koghf)/urdf/turtlebot3_burger.gazebo.xacro"/>
-  <link name="base_footprint"/>
+ <link name="base_footprint"/>
   <joint name="base_joint" type="fixed">
     <parent link="base_footprint"/>
     <child link="base_link"/>
-    <origin xyz="0.0 0.0 0.010" rpy="0 0 0"/>
+    <origin xyz="0.0 0.0 0.0" rpy="0 0 0"/>
   </joint>
   <link name="base_link">
     <visual>
-      <origin xyz="-0.032 0 0.0" rpy="0 0 0"/>
-      <geometry>
-        <mesh filename="package://koghf/meshes/bases/burger_base.stl" scale="0.001 0.001 0.005"/>
-      </geometry>
-      <material name="light_black"/>
-    </visual>
-    <collision>
-      <origin xyz="-0.032 0 0.070" rpy="0 0 0"/>
-      <geometry>
-        <box size="0.140 0.140 0.143"/>
-      </geometry>
-    </collision>
-    <inertial>
-      <origin xyz="0 0 0" rpy="0 0 0"/>
-      <mass value="8.2573504e-01"/>
-      <inertia ixx="2.2124416e-03" ixy="-1.2294101e-05" ixz="3.4938785e-05"
-               iyy="2.1193702e-03" iyz="-5.0120904e-06"
-               izz="2.0064271e-03" />
+      <origin xyz="0 0 0.57" rpy="0 0 0"/>
+      <geometry>
+        <cylinder length="1" radius="0.20"/>
+      </geometry>
+    </visual>
+    <collision>
+      <origin xyz="0 0 0.57" rpy="0 0 0"/>
+      <geometry>
+        <cylinder length="1" radius="0.17"/>
+      </geometry>
+    </collision>
+    <inertial>
+      <origin xyz="0 0 0.57" rpy="0 0 0"/>
+      <mass value="10"/>
+      <inertia ixx=" 1.266667 " ixy="0" ixz="0"
+               iyy=" 1.266667 " iyz="0"
+               izz="0.3" />
     </inertial>
   </link>
@@ -34,5 +33,5 @@
     <parent link="base_link"/>
     <child link="wheel_left_link"/>
-    <origin xyz="0.0 0.08 0.023" rpy="-1.57 0 0"/>
+    <origin xyz="0.12 0.23 0.165" rpy="-1.57 0 0"/>
     <axis xyz="0 0 1"/>
   </joint>
@@ -41,5 +40,5 @@
       <origin xyz="0 0 0" rpy="1.57 0 0"/>
       <geometry>
-        <mesh filename="package://koghf/meshes/wheels/left_tire.stl" scale="0.001 0.001 0.001"/>
+        <mesh filename="package://koghf/meshes/wheels/left_tire.stl" scale="0.005 0.005 0.005"/>
       </geometry>
       <material name="dark"/>
@@ -48,13 +47,13 @@
       <origin xyz="0 0 0" rpy="0 0 0"/>
       <geometry>
-        <cylinder length="0.018" radius="0.033"/>
-      </geometry>
-    </collision>
-    <inertial>
-      <origin xyz="0 0 0" />
-      <mass value="2.8498940e-02" />
-      <inertia ixx="1.1175580e-05" ixy="-4.2369783e-11" ixz="-5.9381719e-09"
-               iyy="1.1192413e-05" iyz="-1.4400107e-11"
-               izz="2.0712558e-05" />
+        <cylinder length="0.09" radius="0.165"/>
+      </geometry>
+    </collision>
+    <inertial>
+      <origin xyz="0 0 0" />
+      <mass value="10.5498940" />
+      <inertia ixx="0.021321" ixy="0" ixz="0"
+               iyy="0.021321" iyz="0"
+               izz="0.038794 " />
       </inertial>
   </link>
@@ -62,5 +61,5 @@
     <parent link="base_link"/>
     <child link="wheel_right_link"/>
-    <origin xyz="0.0 -0.080 0.023" rpy="-1.57 0 0"/>
+    <origin xyz="0.12 -0.23 0.165" rpy="-1.57 0 0"/>
     <axis xyz="0 0 1"/>
   </joint>
@@ -69,5 +68,5 @@
       <origin xyz="0 0 0" rpy="1.57 0 0"/>
       <geometry>
-        <mesh filename="package://koghf/meshes/wheels/right_tire.stl" scale="0.001 0.001 0.001"/>
+        <mesh filename="package://koghf/meshes/wheels/right_tire.stl" scale="0.005 0.005 0.005"/>
       </geometry>
       <material name="dark"/>
@@ -76,13 +75,13 @@
       <origin xyz="0 0 0" rpy="0 0 0"/>
       <geometry>
-        <cylinder length="0.018" radius="0.033"/>
-      </geometry>
-    </collision>
-    <inertial>
-      <origin xyz="0 0 0" />
-      <mass value="2.8498940e-02" />
-      <inertia ixx="1.1175580e-05" ixy="-4.2369783e-11" ixz="-5.9381719e-09"
-               iyy="1.1192413e-05" iyz="-1.4400107e-11"
-               izz="2.0712558e-05" />
+        <cylinder length="0.09" radius="0.165"/>
+      </geometry>
+    </collision>
+    <inertial>
+      <origin xyz="0 0 0" />
+      <mass value="10.5498940" />
+      <inertia ixx="0.021321" ixy="0" ixz="0"
+               iyy="0.021321" iyz="0"
+               izz="0.038794" />
       </inertial>
   </link>
@@ -90,11 +89,17 @@
     <parent link="base_link"/>
     <child link="caster_back_link"/>
-    <origin xyz="-0.081 0 -0.004" rpy="-1.57 0 0"/>
+    <origin xyz="-0.22 0 0.022" rpy="-1.57 0 0"/>
   </joint>
   <link name="caster_back_link">
-    <collision>
-      <origin xyz="0 0.001 0" rpy="0 0 0"/>
-      <geometry>
-        <box size="0.030 0.009 0.020"/>
+    <visual>
+      <origin xyz="0 0 0" rpy="0 0 1.57"/>
+      <geometry>
+       <cylinder length = "0.05" radius = "0.02" />
+      </geometry>
+    </visual>
+    <collision>
+      <origin xyz="0 0 0" rpy="0 0 0"/>
+      <geometry>
+       <cylinder length = "0.05" radius = "0.02" />
       </geometry>
     </collision>
@@ -141,6 +146,6 @@
   </link>
   <!-- Camera -->
-  <joint type="fixed" name="camera_joint">
-    <origin xyz="-0.03 0 0.81" rpy="0 -1.5708 0"/>
+  <joint type="continuous" name="camera_joint">
+    <origin xyz="0 0 1.08" rpy="0 -1.5708 0"/>
     <child link="camera_link"/>
     <parent link="base_link"/>
@@ -174,4 +179,7 @@
     <material>Gazebo/Red</material>
   </gazebo>
+   <gazebo reference="caster_back_link">
+    <material>Gazebo/Grey</material>
+  </gazebo>
   <joint type="fixed" name="camera_optical_joint">
     <origin xyz="0 0 0" rpy="-1.5707 0 -1.5707"/>
@@ -181,3 +189,34 @@
   <link name="camera_link_optical">
   </link>
+ <!-- Tray -->
+  <joint type="fixed" name="tray_joint">
+    <origin xyz="0 0 1.075" rpy="0 0 -1.5708"/>
+    <child link="tray_link"/>
+    <parent link="base_link"/>
+    <axis xyz="0 1 0" />
+  </joint>
+  <link name='tray_link'>
+    <pose>0 0 0 0 0 0</pose>
+    <visual>
+      <origin xyz="0 0 0" rpy="0 0 0"/>
+      <geometry>
+        <mesh filename="package://koghf/meshes/coffee_tray.stl" scale="0.013 0.016 0.013"/>
+      </geometry>
+    </visual>
+    <visual>
+      <origin xyz="0 0 0" rpy="0 0 0"/>
+      <geometry>
+        <box size=".39 .38 .007" />
+      </geometry>
+    </visual>
+    <inertial>
+      <mass value="0.01"/>
+      <origin xyz="0 0 0" rpy="0 0 0"/>
+      <inertia
+          ixx="1e-6" ixy="0" ixz="0"
+          iyy="1e-6" iyz="0"
+          izz="1e-6"
+      />
+    </inertial>
+  </link>
 </robot>

Commit message: működőképes + video

File: urdf/turtlebot3_burger.gazebo.xacro (robot description, xacro)
@@ -10,6 +10,6 @@
   </gazebo>
   <gazebo reference="wheel_left_link">
-    <mu1>50</mu1>
-    <mu2>50</mu2>
+    <mu1>3</mu1>
+    <mu2>0.55</mu2>
     <kp>500000.0</kp>
     <kd>10.0</kd>
@@ -20,6 +20,6 @@
   </gazebo>
   <gazebo reference="wheel_right_link">
-    <mu1>50</mu1>
-    <mu2>50</mu2>
+    <mu1>3</mu1>
+    <mu2>0.55</mu2>
     <kp>500000.0</kp>
     <kd>10.0</kd>
@@ -30,11 +30,11 @@
   </gazebo>
   <gazebo reference="caster_back_link">
-    <mu1>0.01</mu1>
-    <mu2>0.01</mu2>
+    <mu1>0.1</mu1>
+    <mu2>0.1</mu2>
     <kp>1000000.0</kp>
     <kd>100.0</kd>
     <minDepth>0.001</minDepth>
     <maxVel>1.0</maxVel>
-    <material>Gazebo/</material>
+    <material>Gazebo/FlatBlack</material>
   </gazebo>
   <gazebo reference="imu_link">
@@ -46,5 +46,5 @@
   </gazebo>
   <gazebo>
-    <plugin name="turtlebot3_burger_controller" filename="libgazebo_ros_diff_drive.so">
+    <plugin name="differential_drive_controller" filename="libgazebo_ros_diff_drive.so">
       <commandTopic>cmd_vel</commandTopic>
       <odometryTopic>odom</odometryTopic>
@@ -57,11 +57,11 @@
       <publishWheelJointState>true</publishWheelJointState>
       <legacyMode>false</legacyMode>
-      <updateRate>600</updateRate>
+      <updateRate>120</updateRate>
       <leftJoint>wheel_left_joint</leftJoint>
       <rightJoint>wheel_right_joint</rightJoint>
       <wheelSeparation>0.46</wheelSeparation>
       <wheelDiameter>0.33</wheelDiameter>
-      <wheelAcceleration>3</wheelAcceleration>
-      <wheelTorque>10</wheelTorque>
+      <wheelAcceleration>1</wheelAcceleration>
+      <wheelTorque>20</wheelTorque>
       <rosDebugLevel>na</rosDebugLevel>
     </plugin>

File: urdf/turtlebot3_burger.xacro (robot description, xacro)
@@ -24,7 +24,7 @@
     <inertial>
       <origin xyz="0 0 0.57" rpy="0 0 0"/>
-      <mass value="10"/>
-      <inertia ixx=" 1.266667 " ixy="0" ixz="0"
-               iyy=" 1.266667 " iyz="0"
+      <mass value="15"/>
+      <inertia ixx=" 1.296667 " ixy="0" ixz="0"
+               iyy=" 1.296667 " iyz="0"
                izz="0.3" />
     </inertial>
@@ -33,5 +33,5 @@
     <parent link="base_link"/>
     <child link="wheel_left_link"/>
-    <origin xyz="0.12 0.23 0.165" rpy="-1.57 0 0"/>
+    <origin xyz="0.15 0.23 0.165" rpy="-1.57 0 0"/>
     <axis xyz="0 0 1"/>
   </joint>
@@ -52,5 +52,5 @@
     <inertial>
       <origin xyz="0 0 0" />
-      <mass value="10.5498940" />
+      <mass value="2.5498940" />
       <inertia ixx="0.021321" ixy="0" ixz="0"
                iyy="0.021321" iyz="0"
@@ -61,5 +61,5 @@
     <parent link="base_link"/>
     <child link="wheel_right_link"/>
-    <origin xyz="0.12 -0.23 0.165" rpy="-1.57 0 0"/>
+    <origin xyz="0.15 -0.23 0.165" rpy="-1.57 0 0"/>
     <axis xyz="0 0 1"/>
   </joint>
@@ -80,5 +80,5 @@
     <inertial>
       <origin xyz="0 0 0" />
-      <mass value="10.5498940" />
+      <mass value="2.5498940" />
       <inertia ixx="0.021321" ixy="0" ixz="0"
                iyy="0.021321" iyz="0"
@@ -95,11 +95,11 @@
       <origin xyz="0 0 0" rpy="0 0 1.57"/>
       <geometry>
-       <cylinder length = "0.05" radius = "0.02" />
-      </geometry>
-    </visual>
-    <collision>
-      <origin xyz="0 0 0" rpy="0 0 0"/>
-      <geometry>
-       <cylinder length = "0.05" radius = "0.02" />
+        <sphere radius="0.02"/>
+      </geometry>
+    </visual>
+    <collision>
+      <origin xyz="0 0 0" rpy="0 0 0"/>
+      <geometry>
+      <sphere radius="0.02"/>
       </geometry>
     </collision>
